File: Schematic/final_project.sch (EAGLE design)
At the start: 6 parts

Commit message: Finished schematic
Parts:
- removed FEEDBACK_RESISTOR: 1K, resistor:R-US_0204/2V
- added FEEDBACK: 1K, resistor:R-US_0204/2V
Connections:
- removed net N$1: FEEDBACK_RESISTOR.1, U$1.AC1RX/*SS3A/U3BRX/*U3ACTS/RF12, VGA_HEADER.13
- new net GND: CLAMPING_DIODE.C, PS/2_HEADER.3, VGA_HEADER.5, VGA_HEADER.6, VGA_HEADER.7, VGA_HEADER.8, VGA_HEADER.9
- new net N$10: FEEDBACK.2, U$1.AC1RX/*SS3A/U3BRX/*U3ACTS/RF12
- new net VCC: PS/2_HEADER.4
- net N$7: now also FEEDBACK.1, VGA_HEADER.13; no longer FEEDBACK_RESISTOR.2
Other:
- moved on the sheet: COLOR_JUMPERS, VGA_HEADER
Changed lines of the file:
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@@
 <parts>
 <part name="CLAMPING_DIODE" library="diode" deviceset="1N4004" device="" value="1N4148"/>
-<part name="FEEDBACK_RESISTOR" library="resistor" deviceset="R-US_" device="0204/2V" value="1K"/>
+<part name="FEEDBACK" library="resistor" deviceset="R-US_" device="0204/2V" value="1K"/>
 <part name="VGA_HEADER" library="con-subd" deviceset="HF15" device="H"/>
 <part name="PS/2_HEADER" library="con-yamaichi" deviceset="MDIN06K" device=""/>
 <part name="U$1" library="PIC32MX795F512L" deviceset="PIC32MX795F512L-X_PF" device=""/>
 <part name="COLOR_JUMPERS" library="jumper" deviceset="JP3Q" device=""/>
+<part name="GND1" library="supply1" deviceset="GND" device=""/>
+<part name="GND2" library="supply1" deviceset="GND" device=""/>
+<part name="P+2" library="supply1" deviceset="VCC" device=""/>
+<part name="FRAME1" library="frames" deviceset="DINA3_L" device=""/>
 </parts>
 <sheets>
@@
 <instances>
 <instance part="CLAMPING_DIODE" gate="1" x="330.2" y="-40.64"/>
-<instance part="FEEDBACK_RESISTOR" gate="G$1" x="45.72" y="-10.16"/>
-<instance part="VGA_HEADER" gate="G$1" x="393.7" y="-30.48"/>
+<instance part="FEEDBACK" gate="G$1" x="45.72" y="2.54"/>
+<instance part="VGA_HEADER" gate="G$1" x="373.38" y="-30.48"/>
 <instance part="PS/2_HEADER" gate="G$1" x="393.7" y="10.16"/>
 <instance part="U$1" gate="A" x="63.5" y="25.4"/>
-<instance part="COLOR_JUMPERS" gate="B" x="368.3" y="-25.4" rot="R90"/>
+<instance part="COLOR_JUMPERS" gate="B" x="342.9" y="-25.4" rot="R90"/>
+<instance part="GND1" gate="1" x="381" y="0"/>
+<instance part="GND2" gate="1" x="350.52" y="-73.66"/>
+<instance part="P+2" gate="VCC" x="378.46" y="27.94"/>
+<instance part="FRAME1" gate="G$1" x="22.86" y="-190.5"/>
+<instance part="FRAME1" gate="G$2" x="309.88" y="-190.5"/>
 </instances>
 <busses>
 </busses>
 <nets>
-<net name="N$1" class="0">
-<segment>
-<pinref part="U$1" gate="A" pin="AC1RX/*SS3A/U3BRX/*U3ACTS/RF12"/>
-<wire x1="63.5" y1="20.32" x2="40.64" y2="20.32" width="0.1524" layer="91"/>
-<wire x1="40.64" y1="20.32" x2="40.64" y2="-10.16" width="0.1524" layer="91"/>
-<pinref part="FEEDBACK_RESISTOR" gate="G$1" pin="1"/>
-<wire x1="40.64" y1="-10.16" x2="40.64" y2="-119.38" width="0.1524" layer="91"/>
-<junction x="40.64" y="-10.16"/>
-<wire x1="40.64" y1="-119.38" x2="429.26" y2="-119.38" width="0.1524" layer="91"/>
-<wire x1="429.26" y1="-119.38" x2="429.26" y2="-30.48" width="0.1524" layer="91"/>
-<wire x1="429.26" y1="-30.48" x2="401.32" y2="-30.48" width="0.1524" layer="91"/>
-<pinref part="VGA_HEADER" gate="G$1" pin="13"/>
-</segment>
-</net>
 <net name="N$2" class="0">
 <segment>
 <pinref part="COLOR_JUMPERS" gate="B" pin="5"/>
 <pinref part="VGA_HEADER" gate="G$1" pin="1"/>
-<wire x1="375.92" y1="-22.86" x2="386.08" y2="-20.32" width="0.1524" layer="91"/>
+<wire x1="350.52" y1="-22.86" x2="365.76" y2="-20.32" width="0.1524" layer="91"/>
 </segment>
 </net>
@@
 <pinref part="COLOR_JUMPERS" gate="B" pin="3"/>
 <pinref part="VGA_HEADER" gate="G$1" pin="2"/>
-<wire x1="375.92" y1="-25.4" x2="386.08" y2="-25.4" width="0.1524" layer="91"/>
+<wire x1="350.52" y1="-25.4" x2="365.76" y2="-25.4" width="0.1524" layer="91"/>
 </segment>
 </net>
@@
 <pinref part="COLOR_JUMPERS" gate="B" pin="1"/>
 <pinref part="VGA_HEADER" gate="G$1" pin="3"/>
-<wire x1="375.92" y1="-27.94" x2="386.08" y2="-30.48" width="0.1524" layer="91"/>
+<wire x1="350.52" y1="-27.94" x2="365.76" y2="-30.48" width="0.1524" layer="91"/>
 </segment>
 </net>
@@
 <pinref part="COLOR_JUMPERS" gate="B" pin="6"/>
 <pinref part="COLOR_JUMPERS" gate="B" pin="4"/>
-<wire x1="360.68" y1="-22.86" x2="360.68" y2="-25.4" width="0.1524" layer="91"/>
+<wire x1="335.28" y1="-22.86" x2="335.28" y2="-25.4" width="0.1524" layer="91"/>
 <pinref part="COLOR_JUMPERS" gate="B" pin="2"/>
-<wire x1="360.68" y1="-27.94" x2="360.68" y2="-25.4" width="0.1524" layer="91"/>
-<junction x="360.68" y="-25.4"/>
-<wire x1="360.68" y1="-25.4" x2="327.66" y2="-25.4" width="0.1524" layer="91"/>
+<wire x1="335.28" y1="-27.94" x2="335.28" y2="-25.4" width="0.1524" layer="91"/>
+<junction x="335.28" y="-25.4"/>
+<wire x1="335.28" y1="-25.4" x2="327.66" y2="-25.4" width="0.1524" layer="91"/>
 <pinref part="CLAMPING_DIODE" gate="1" pin="A"/>
 <wire x1="327.66" y1="-25.4" x2="327.66" y2="-40.64" width="0.1524" layer="91"/>
@@
 <net name="N$7" class="0">
 <segment>
-<pinref part="FEEDBACK_RESISTOR" gate="G$1" pin="2"/>
-<wire x1="50.8" y1="-10.16" x2="50.8" y2="-33.02" width="0.1524" layer="91"/>
-<wire x1="50.8" y1="-33.02" x2="63.5" y2="-33.02" width="0.1524" layer="91"/>
+<wire x1="40.64" y1="-33.02" x2="63.5" y2="-33.02" width="0.1524" layer="91"/>
+<pinref part="FEEDBACK" gate="G$1" pin="1"/>
+<wire x1="40.64" y1="-33.02" x2="40.64" y2="2.54" width="0.1524" layer="91"/>
+<wire x1="40.64" y1="-119.38" x2="388.62" y2="-116.84" width="0.1524" layer="91"/>
+<wire x1="388.62" y1="-116.84" x2="388.62" y2="-30.48" width="0.1524" layer="91"/>
+<wire x1="388.62" y1="-30.48" x2="381" y2="-30.48" width="0.1524" layer="91"/>
+<pinref part="VGA_HEADER" gate="G$1" pin="13"/>
+<wire x1="40.64" y1="-33.02" x2="40.64" y2="-119.38" width="0.1524" layer="91"/>
+<junction x="40.64" y="-33.02"/>
 </segment>
 </net>
@@
 <segment>
 <pinref part="U$1" gate="A" pin="AN8/C1OUT/RB8"/>
-<wire x1="63.5" y1="-27.94" x2="30.48" y2="-27.94" width="0.1524" layer="91"/>
-<wire x1="30.48" y1="-27.94" x2="30.48" y2="-132.08" width="0.1524" layer="91"/>
-<wire x1="30.48" y1="-132.08" x2="441.96" y2="-132.08" width="0.1524" layer="91"/>
-<wire x1="441.96" y1="-132.08" x2="441.96" y2="-35.56" width="0.1524" layer="91"/>
+<wire x1="63.5" y1="-27.94" x2="35.56" y2="-27.94" width="0.1524" layer="91"/>
+<wire x1="35.56" y1="-27.94" x2="35.56" y2="-132.08" width="0.1524" layer="91"/>
+<wire x1="35.56" y1="-132.08" x2="398.78" y2="-129.54" width="0.1524" layer="91"/>
+<wire x1="398.78" y1="-129.54" x2="398.78" y2="-35.56" width="0.1524" layer="91"/>
 <pinref part="VGA_HEADER" gate="G$1" pin="14"/>
-<wire x1="441.96" y1="-35.56" x2="401.32" y2="-35.56" width="0.1524" layer="91"/>
+<wire x1="398.78" y1="-35.56" x2="381" y2="-35.56" width="0.1524" layer="91"/>
 </segment>
 </net>
@@
 </segment>
 </net>
+<net name="N$10" class="0">
+<segment>
+<pinref part="U$1" gate="A" pin="AC1RX/*SS3A/U3BRX/*U3ACTS/RF12"/>
+<wire x1="63.5" y1="20.32" x2="55.88" y2="20.32" width="0.1524" layer="91"/>
+<pinref part="FEEDBACK" gate="G$1" pin="2"/>
+<wire x1="50.8" y1="2.54" x2="55.88" y2="2.54" width="0.1524" layer="91"/>
+<wire x1="55.88" y1="2.54" x2="55.88" y2="20.32" width="0.1524" layer="91"/>
+</segment>
+</net>
+<net name="GND" class="0">
+<segment>
+<pinref part="CLAMPING_DIODE" gate="1" pin="C"/>
+<pinref part="GND2" gate="1" pin="GND"/>
+<wire x1="332.74" y1="-40.64" x2="350.52" y2="-40.64" width="0.1524" layer="91"/>
+<wire x1="350.52" y1="-40.64" x2="350.52" y2="-71.12" width="0.1524" layer="91"/>
+<pinref part="VGA_HEADER" gate="G$1" pin="5"/>
+<wire x1="365.76" y1="-40.64" x2="363.22" y2="-40.64" width="0.1524" layer="91"/>
+<junction x="350.52" y="-40.64"/>
+<pinref part="VGA_HEADER" gate="G$1" pin="6"/>
+<wire x1="363.22" y1="-40.64" x2="360.68" y2="-40.64" width="0.1524" layer="91"/>
+<wire x1="360.68" y1="-40.64" x2="358.14" y2="-40.64" width="0.1524" layer="91"/>
+<wire x1="358.14" y1="-40.64" x2="355.6" y2="-40.64" width="0.1524" layer="91"/>
+<wire x1="355.6" y1="-40.64" x2="350.52" y2="-40.64" width="0.1524" layer="91"/>
+<wire x1="365.76" y1="-22.86" x2="355.6" y2="-22.86" width="0.1524" layer="91"/>
+<wire x1="355.6" y1="-22.86" x2="355.6" y2="-40.64" width="0.1524" layer="91"/>
+<junction x="355.6" y="-40.64"/>
+<pinref part="VGA_HEADER" gate="G$1" pin="7"/>
+<wire x1="365.76" y1="-27.94" x2="358.14" y2="-27.94" width="0.1524" layer="91"/>
+<wire x1="358.14" y1="-27.94" x2="358.14" y2="-40.64" width="0.1524" layer="91"/>
+<junction x="358.14" y="-40.64"/>
+<pinref part="VGA_HEADER" gate="G$1" pin="8"/>
+<wire x1="365.76" y1="-33.02" x2="360.68" y2="-33.02" width="0.1524" layer="91"/>
+<wire x1="360.68" y1="-33.02" x2="360.68" y2="-40.64" width="0.1524" layer="91"/>
+<junction x="360.68" y="-40.64"/>
+<pinref part="VGA_HEADER" gate="G$1" pin="9"/>
+<wire x1="365.76" y1="-38.1" x2="363.22" y2="-38.1" width="0.1524" layer="91"/>
+<wire x1="363.22" y1="-38.1" x2="363.22" y2="-40.64" width="0.1524" layer="91"/>
+<junction x="363.22" y="-40.64"/>
+</segment>
+<segment>
+<pinref part="PS/2_HEADER" gate="G$1" pin="3"/>
+<pinref part="GND1" gate="1" pin="GND"/>
+<wire x1="386.08" y1="12.7" x2="381" y2="12.7" width="0.1524" layer="91"/>
+<wire x1="381" y1="12.7" x2="381" y2="2.54" width="0.1524" layer="91"/>
+</segment>
+</net>
+<net name="VCC" class="0">
+<segment>
+<pinref part="PS/2_HEADER" gate="G$1" pin="4"/>
+<pinref part="P+2" gate="VCC" pin="VCC"/>
+<wire x1="386.08" y1="10.16" x2="378.46" y2="10.16" width="0.1524" layer="91"/>
+<wire x1="378.46" y1="10.16" x2="378.46" y2="25.4" width="0.1524" layer="91"/>
+</segment>
+</net>
